File: pcb/03_motor_control_inverter.kicad_sch (KiCad schematic)
At the start: 0 parts

Commit message: Unified all different LCSC part numbers of the same exact components to just one variant
Parts:
- added C801, C802, C805, C806, C809, C810: 3n3 10% 100V, FluxNode-FOC:C_0402_1005_DensityHigh, symbol Device:C
- added C803, C808, C812: 4.7u 100V, FluxNode-FOC:C_1206_3216_DensityHigh, symbol Device:C
- added C804, C807, C811: 100nF 100V, FluxNode-FOC:C_1206_3216_DensityHigh, symbol Device:C
- added D801, D802, D803, D804, D805, D806, D807, D808, D809: BAT41ZFILM, FluxNode-FOC:SOD3816X145N, symbol FluxNode-FOC:BAT41ZFILM
- added NT801: SRC_HS_A, symbol Device:NetTie_2
- added NT802: SHUNT_P_A, symbol Device:NetTie_2
- added NT803: SHUNT_L_A, symbol Device:NetTie_2
- added NT804: SRC_HS_B, symbol Device:NetTie_2
- added NT805: SHUNT_P_B, symbol Device:NetTie_2
- added NT806: SHUNT_L_B, symbol Device:NetTie_2
- added NT807: SRC_HS_C, symbol Device:NetTie_2
- added NT808: SHUNT_P_C, symbol Device:NetTie_2
- added NT809: SHUNT_L_C, symbol Device:NetTie_2
- added Q801, Q802, Q803, Q804, Q805, Q806: TPW1R306PL, FluxNode-FOC:SOP_ADVANCE, symbol FluxNode-FOC:TPW1R306PL
- added R801, R802, R815, R816, R820, R821: 7.5 1% 0.5W, FluxNode-FOC:R_0805_2012_DensityHigh, symbol Device:R
- added R803, R804, R818, R819, R823, R824: 5R 1% 0.4W, FluxNode-FOC:R_0603_1608_DensityHigh, symbol Device:R
- added R805, R817, R822: 0.5m 1% 2W, FluxNode-FOC:R_1206_3216_DensityHigh, symbol Device:R
- added R806, R807, R809, R810, R812, R813: 51k 1% 75V, FluxNode-FOC:R_0603_1608_DensityHigh, symbol Device:R
- added R808, R811, R814: 6k8 1% 75V, FluxNode-FOC:R_0603_1608_DensityHigh, symbol Device:R
Connections:
- new net: R806.1, R807.2
- new net: R809.1, R810.2
- new net: R812.1, R813.2
- new net +VBAT: C803.1, C804.1, C807.1, C808.1, C811.1, C812.1, Q801.5 (D), Q801.6 (D), Q801.7 (D), Q801.8 (D), Q803.5 (D), Q803.6 (D), Q803.7 (D), Q803.8 (D), Q805.5 (D), Q805.6 (D), Q805.7 (D), Q805.8 (D), R803.2, R818.2, R823.2
- new net FET_GH_A: D803.2 (A), Q801.4 (G), R801.2
- new net FET_GH_B: D805.2 (A), Q803.4 (G), R815.2
- new net FET_GH_C: D808.2 (A), Q805.4 (G), R820.2
- new net FET_GL_A: D801.1 (K), D802.2 (A), Q802.4 (G), R802.2
- new net FET_GL_B: D804.1 (K), D806.2 (A), Q804.4 (G), R816.2
- new net FET_GL_C: D807.1 (K), D809.2 (A), Q806.4 (G), R821.2
- new net GATE_HS_A: D803.1 (K), R801.1
- new net GATE_HS_B: D805.1 (K), R815.1
- new net GATE_HS_C: D808.1 (K), R820.1
- new net GATE_LS_A: D802.1 (K), R802.1
- new net GATE_LS_B: D806.1 (K), R816.1
- new net GATE_LS_C: D809.1 (K), R821.1
- new net GND: C803.2, C808.2, C812.2, D801.2 (A), D804.2 (A), D807.2 (A), NT803.2, NT806.2, NT809.2, R805.1, R808.1, R811.1, R814.1, R817.1, R822.1
- new net PHA: C801.2, C802.2, NT801.2, Q801.1 (S), Q801.2 (S), Q801.3 (S), Q802.5 (D), Q802.6 (D), Q802.7 (D), Q802.8 (D), R806.2
- new net PHB: C805.2, C806.2, NT804.2, Q803.1 (S), Q803.2 (S), Q803.3 (S), Q804.5 (D), Q804.6 (D), Q804.7 (D), Q804.8 (D), R809.2
- new net PHC: C809.2, C810.2, NT807.2, Q805.1 (S), Q805.2 (S), Q805.3 (S), Q806.5 (D), Q806.6 (D), Q806.7 (D), Q806.8 (D), R812.2
- new net SENSE_UA: R807.1, R808.2
- new net SENSE_UB: R810.1, R811.2
- new net SENSE_UC: R813.1, R814.2
- new net SHUNT_N_A: NT803.1
- new net SHUNT_N_B: NT806.1
- new net SHUNT_N_C: NT809.1
- new net SHUNT_P_A: NT802.1
- new net SHUNT_P_B: NT805.1
- new net SHUNT_P_C: NT808.1
- new net SNUB_HA: C801.1, R803.1
- new net SNUB_HB: C805.1, R818.1
- new net SNUB_HC: C809.1, R823.1
- new net SNUB_LA: C802.1, R804.1
- new net SNUB_LB: C806.1, R819.1
- new net SNUB_LC: C810.1, R824.1
- new net SRC_HS_A: NT801.1
- new net SRC_HS_B: NT804.1
- new net SRC_HS_C: NT807.1
- new net SRC_LS_A: C804.2, NT802.2, Q802.1 (S), Q802.2 (S), Q802.3 (S), R804.2, R805.2
- new net SRC_LS_B: C807.2, NT805.2, Q804.1 (S), Q804.2 (S), Q804.3 (S), R817.2, R819.2
- new net SRC_LS_C: C811.2, NT808.2, Q806.1 (S), Q806.2 (S), Q806.3 (S), R822.2, R824.2
Other:
- company: (none) -> PhiMai
