File: pcb/04_sensing_position.kicad_sch (KiCad schematic)
At the start: 0 parts

Commit message: Unified all different LCSC part numbers of the same exact components to just one variant
Other:
- company: (none) -> PhiMai
Changed lines of the file:
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@@
 	(generator_version "10.0")
 	(paper "A4")
+	(title_block
+		(date "2026-06-07")
+		(rev "0.1.0")
+		(company "PhiMai")
+	)
+	(hierarchical_label "{SPI1_MAG}"
+		(shape bidirectional)
+		(at 125.73 69.85 0)
+		(effects
+			(font
+				(size 1.27 1.27)
+			)
+			(justify left)
+		)
+	)
 )
