File: hardware/kicad/FluxNode-FOC.kicad_sch (KiCad schematic)
At the start: 0 parts

Commit message: Reorganised pdb folder structure to acomodate seperate sheets folder and an erxternal lib folder
Other:
- sheet 01 Power Connectors: file 01_power_connectors.kicad_sch -> sheets/01_power_connectors.kicad_sch
- sheet 01 Power Generation: file 01_power_generation.kicad_sch -> sheets/01_power_generation.kicad_sch
- sheet 02 MCU: file 02-mcu.kicad_sch -> sheets/02-mcu.kicad_sch
- sheet 03 Motor Control - Brake Chopper: file 03_motor_control_brake_chopper.kicad_sch -> sheets/03_motor_control_brake_chopper.kicad_sch
- sheet 03 Motor Control - Gate Driver: file 03_motor_control_gate_driver.kicad_sch -> sheets/03_motor_control_gate_driver.kicad_sch
- sheet 04 Sensing - Battery: file 04_sensing_battery.kicad_sch -> sheets/04_sensing_battery.kicad_sch
- sheet 04 Sensing - Position: file 04_sensing_position.kicad_sch -> sheets/04_sensing_position.kicad_sch
- sheet 04 Sensing - Temp: file 04_sensing_temp.kicad_sch -> sheets/04_sensing_temp.kicad_sch
- sheet 05 Interface - FD CAN: file 05_interface_fd_can.kicad_sch -> sheets/05_interface_fd_can.kicad_sch
- sheet 05 Interface - Fan Control: file 05_interface_fan_control.kicad_sch -> sheets/05_interface_fan_control.kicad_sch
- sheet 05 Interface - Interconnects: file 05_interface_interconnects.kicad_sch -> sheets/05_interface_interconnects.kicad_sch
- sheet 06 User - LED Indicators: file 06_user_led_indicators.kicad_sch -> sheets/06_user_led_indicators.kicad_sch
- sheet 07 Misc - Holes: file 07_misc.kicad_sch -> sheets/07_misc.kicad_sch
Changed lines of the file:
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@@
 			)
 		)
-		(property "Sheetfile" "05_interface_fan_control.kicad_sch"
+		(property "Sheetfile" "sheets/05_interface_fan_control.kicad_sch"
 			(at 72.39 188.5446 0)
 			(show_name no)
@@
 			)
 		)
-		(property "Sheetfile" "02-mcu.kicad_sch"
+		(property "Sheetfile" "sheets/02-mcu.kicad_sch"
 			(at 130.81 208.8646 0)
 			(show_name no)
@@
 			)
 		)
-		(property "Sheetfile" "05_interface_fd_can.kicad_sch"
+		(property "Sheetfile" "sheets/05_interface_fd_can.kicad_sch"
 			(at 72.39 172.0346 0)
 			(show_name no)
@@
 			)
 		)
-		(property "Sheetfile" "06_user_led_indicators.kicad_sch"
+		(property "Sheetfile" "sheets/06_user_led_indicators.kicad_sch"
 			(at 185.42 137.7446 0)
 			(show_name no)
@@
 			)
 		)
-		(property "Sheetfile" "01_power_generation.kicad_sch"
+		(property "Sheetfile" "sheets/01_power_generation.kicad_sch"
 			(at 72.39 53.9246 0)
 			(show_name no)
@@
 			)
 		)
-		(property "Sheetfile" "03_motor_control_gate_driver.kicad_sch"
+		(property "Sheetfile" "sheets/03_motor_control_gate_driver.kicad_sch"
 			(at 184.15 88.2146 0)
 			(show_name no)
@@
 			)
 		)
-		(property "Sheetfile" "04_sensing_battery.kicad_sch"
+		(property "Sheetfile" "sheets/04_sensing_battery.kicad_sch"
 			(at 72.39 74.2446 0)
 			(show_name no)
@@
 			)
 		)
-		(property "Sheetfile" "04_sensing_position.kicad_sch"
+		(property "Sheetfile" "sheets/04_sensing_position.kicad_sch"
 			(at 72.39 116.1546 0)
 			(show_name no)
@@
 			)
 		)
-		(property "Sheetfile" "03_motor_control_brake_chopper.kicad_sch"
+		(property "Sheetfile" "sheets/03_motor_control_brake_chopper.kicad_sch"
 			(at 184.15 116.1546 0)
 			(show_name no)
@@
 			)
 		)
-		(property "Sheetfile" "01_power_connectors.kicad_sch"
+		(property "Sheetfile" "sheets/01_power_connectors.kicad_sch"
 			(at 25.4 53.9246 0)
 			(show_name no)
@@
 			)
 		)
-		(property "Sheetfile" "05_interface_interconnects.kicad_sch"
+		(property "Sheetfile" "sheets/05_interface_interconnects.kicad_sch"
 			(at 72.39 155.5246 0)
 			(show_name no)
@@
 			)
 		)
-		(property "Sheetfile" "07_misc.kicad_sch"
+		(property "Sheetfile" "sheets/07_misc.kicad_sch"
 			(at 185.42 155.5246 0)
 			(show_name no)
@@
 			)
 		)
-		(property "Sheetfile" "04_sensing_temp.kicad_sch"
+		(property "Sheetfile" "sheets/04_sensing_temp.kicad_sch"
 			(at 72.39 100.9146 0)
 			(show_name no)
