File: hardware/kicad/sheets/03_motor_control_gate_driver.kicad_sch (KiCad schematic)
At the start: 11 parts, among them IC1 DRV8323SRTAR

Commit message: Reorganised pdb folder structure to acomodate seperate sheets folder and an erxternal lib folder
Other:
- sheet 03 Motor Control - Inverter: file 03_motor_control_inverter.kicad_sch -> sheets/03_motor_control_inverter.kicad_sch
Changed lines of the file:
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@@
 			)
 		)
-		(property "Sheetfile" "03_motor_control_inverter.kicad_sch"
+		(property "Sheetfile" "sheets/03_motor_control_inverter.kicad_sch"
 			(at 138.43 126.3146 0)
 			(show_name no)
