File: hardware/kicad/sheets/sheets/03_motor_control_inverter.kicad_sch (KiCad schematic)
At the start: 60 parts, among them Q801 TPW1R306PL, Q802 TPW1R306PL, Q803 TPW1R306PL, Q804 TPW1R306PL, Q805 TPW1R306PL, Q806 TPW1R306PL

Commit message: Reorganised pdb folder structure to acomodate seperate sheets folder and an erxternal lib folder
Parts:
- renumbered C808 to C?, C810 to C?, C806 to C?, C801 to C?, C803 to C?, C802 to C?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
